Commit message: ros2 control implementation success

File: arm_ws/src/arm_description/urdf/arm.urdf.xacro (robot description, xacro)
@@ -189,5 +189,5 @@
     </joint>
     <link name="gripper_right">
-        <xacro:default_inertial mass="1.0"/>
+        <xacro:default_inertial mass="0.1"/>
         <visual>
             <origin rpy="0 -1.57 0" xyz="0.0175 0 -0.165"/>
@@ -212,5 +212,5 @@
     </joint>
     <link name="gripper_left">
-        <xacro:default_inertial mass="1.0"/>
+        <xacro:default_inertial mass="0.1"/>
         <visual>
             <origin rpy="0 -1.57 0" xyz="0.0175 -0.035 -0.165"/>
@@ -233,5 +233,5 @@
         <origin rpy="0 0 0" xyz="0 0 -0.035"/>
         <mimic joint="joint6" multiplier="-1" />
-        <limit lower="0" upper="1.57" effort="100.0" velocity="10"/>
+        <limit lower="-1.57" upper="0" effort="100.0" velocity="10"/>
     </joint>
     <xacro:default_transmission number="1"/>
